Commit message: holonomic urdf

File: auto_drive/src/holonomic_sim/models/HolonomicUrdf/model.urdf (robot description, URDF)
Before this commit: robot HolonomicUrdf, 8 links, 7 joints
Links:
- link base_link: mass 1.0 -> 114.395; geometry visual box size=1 1 0.5
- link caster_BL: mass 1.0 -> 0.3; geometry collision sphere radius=0.05; visual sphere radius=0.05
- link caster_BR: mass 1.0 -> 0.3; geometry collision sphere radius=0.05; visual sphere radius=0.05
- link caster_FL: mass 1.0 -> 0.3; geometry collision sphere radius=0.05; visual sphere radius=0.05
- link caster_FR: mass 1.0 -> 0.3; geometry collision sphere radius=0.05; visual sphere radius=0.05
- link wheel: mass 1.0 -> 0.0000001; geometry collision cylinder length=0.001 radius=0.2; visual cylinder length=0.001 radius=0.2
- link wheel_base: mass 1.0 -> 0.01
Joints:
- joint caster_BL_joint: origin xyz=-0.5 -0.5 0 rpy=0 0 0 -> xyz=-0.5 -0.5 -0.25 rpy=0 0 0
- joint caster_BR_joint: origin xyz=-0.5 0.5 0 rpy=0 0 0 -> xyz=-0.5 0.5 -0.25 rpy=0 0 0
- joint caster_FL_joint: origin xyz=0.5 -0.5 0 rpy=0 0 0 -> xyz=0.5 -0.5 -0.25 rpy=0 0 0
- joint caster_FR_joint: origin xyz=0.5 0.5 0 rpy=0 0 0 -> xyz=0.5 0.5 -0.25 rpy=0 0 0
- joint wheel_base_joint: origin xyz=0 0 0.3 rpy=0 0 0 -> xyz=0 0 0 rpy=0 0 0
- joint wheel_joint: origin xyz=0 0 -0.3 rpy=0 0 0 -> xyz=0 0 -0.1 rpy=-1.57 0 0

Commit message: success xacro test

File: auto_drive/src/holonomic_sim/models/HolonomicUrdf/model.urdf (robot description, URDF)
Before this commit: robot HolonomicUrdf, 8 links, 7 joints
Links:
- removed link caster_BL
- removed link caster_BR
- removed link caster_FL
- removed link caster_FR
Joints:
- removed joint caster_BL_joint
- removed joint caster_BR_joint
- removed joint caster_FL_joint
- removed joint caster_FR_joint

Commit message: success full xacro

File: auto_drive/src/holonomic_sim/models/HolonomicUrdf/model.urdf (robot description, URDF)
Before this commit: robot HolonomicUrdf, 4 links, 3 joints
Links:
- link base_link: mass 114.395 -> 100.0

File: auto_drive/src/holonomic_sim/models/HolonomicUrdf/model.xacro (robot description, xacro)
@@ -3,5 +3,5 @@
     <link name="base_footprint"/>
     <xacro:property name="base_size" value="1.0"/>
-    <xacro:rectangular_link_macro suffix="base" mass="100.0" width="${base_size}" height="${base_size/2}" depth="${base_size}" if_collision="false"/>
+    <xacro:rectangular_link_macro suffix="base" mass="100" arg="100.0" width="${base_size}" height="${base_size/2}" depth="${base_size}" if_collision="false"/>
     <joint name="base_joint" type="fixed">
         <parent link="base_footprint"/>

File: auto_drive/src/holonomic_sim/models/HolonomicUrdf/model_tx.xacro (robot description, xacro)
@@ -8,5 +8,5 @@
   <link name="base_link">
     <inertial>
-      <mass value="100.0"/>
+      <mass value="100"/>
       <origin rpy="0 0 0" xyz="0 0 0"/>
       <inertia ixx="10.416666666666668" ixy="0.0" ixz="0.0" iyy="10.416666666666668" iyz="0.0" izz="16.666666666666668"/>
@@ -27,7 +27,7 @@
   <link name="wheel_base_link">
     <inertial>
-      <mass value="10.0"/>
+      <mass value="0.01"/>
       <origin rpy="0 0 0" xyz="0 0 0"/>
-      <inertia ixx="0.23333333333333334" ixy="0.0" ixz="0.0" iyy="0.23333333333333334" iyz="0.0" izz="0.44999999999999996"/>
+      <inertia ixx="233333.33333333334" ixy="0.0" ixz="0.0" iyy="233333.33333333334" iyz="0.0" izz="450000.0"/>
     </inertial>
     <visual>
@@ -48,7 +48,7 @@
   <link name="wheel_link">
     <inertial>
-      <mass value="0.0001"/>
+      <mass value="1e-07"/>
       <origin rpy="0 0 0" xyz="0 0 0"/>
-      <inertia ixx="1.0000083333333337e-06" ixy="0.0" ixz="0.0" iyy="1.0000083333333337e-06" iyz="0.0" izz="2.0000000000000003e-06"/>
+      <inertia ixx="1.0000083333333336" ixy="0.0" ixz="0.0" iyy="1.0000083333333336" iyz="0.0" izz="2.0000000000000004"/>
     </inertial>
     <visual>
@@ -75,7 +75,7 @@
   <link name="caster1_link">
     <inertial>
-      <mass value="0.0001"/>
+      <mass value="0.3"/>
       <origin rpy="0 0 0" xyz="0 0 0"/>
-      <inertia ixx="1.0000000000000002e-07" ixy="0.0" ixz="0.0" iyy="1.0000000000000002e-07" iyz="0.0" izz="1.0000000000000002e-07"/>
+      <inertia ixx="3000000.0" ixy="0.0" ixz="0.0" iyy="3000000.0" iyz="0.0" izz="3000000.0"/>
     </inertial>
     <visual>
@@ -101,7 +101,7 @@
   <link name="caster2_link">
     <inertial>
-      <mass value="0.0001"/>
+      <mass value="0.3"/>
       <origin rpy="0 0 0" xyz="0 0 0"/>
-      <inertia ixx="1.0000000000000002e-07" ixy="0.0" ixz="0.0" iyy="1.0000000000000002e-07" iyz="0.0" izz="1.0000000000000002e-07"/>
+      <inertia ixx="3000000.0" ixy="0.0" ixz="0.0" iyy="3000000.0" iyz="0.0" izz="3000000.0"/>
     </inertial>
     <visual>
@@ -127,7 +127,7 @@
   <link name="caster3_link">
     <inertial>
-      <mass value="0.0001"/>
+      <mass value="0.3"/>
       <origin rpy="0 0 0" xyz="0 0 0"/>
-      <inertia ixx="1.0000000000000002e-07" ixy="0.0" ixz="0.0" iyy="1.0000000000000002e-07" iyz="0.0" izz="1.0000000000000002e-07"/>
+      <inertia ixx="3000000.0" ixy="0.0" ixz="0.0" iyy="3000000.0" iyz="0.0" izz="3000000.0"/>
     </inertial>
     <visual>
@@ -153,7 +153,7 @@
   <link name="caster4_link">
     <inertial>
-      <mass value="0.0001"/>
+      <mass value="0.3"/>
       <origin rpy="0 0 0" xyz="0 0 0"/>
-      <inertia ixx="1.0000000000000002e-07" ixy="0.0" ixz="0.0" iyy="1.0000000000000002e-07" iyz="0.0" izz="1.0000000000000002e-07"/>
+      <inertia ixx="3000000.0" ixy="0.0" ixz="0.0" iyy="3000000.0" iyz="0.0" izz="3000000.0"/>
     </inertial>
     <visual>

File: auto_drive/src/holonomic_sim/models/xacro/common.xacro (robot description, xacro)
@@ -1,5 +1,5 @@
 <robot xmlns:xacro="http://ros.org/wiki/xacro">
-    <xacro:macro name="sphere_macro" params="suffix parent mass radius x y z">
-        <xacro:property name="inertia" value="${2/5*mass*radius*radius}"/>
+    <xacro:macro name="sphere_macro" params="suffix parent mass arg radius x y z">
+        <xacro:property name="inertia" value="${2/5*arg*radius*radius}"/>
         <link name="${suffix}_link">
             <inertial>
@@ -29,5 +29,5 @@
         </joint>
     </xacro:macro>
-    <xacro:macro name="wheel_link_macro" params="suffix mass radius length if_collision">
+    <xacro:macro name="wheel_link_macro" params="suffix mass arg radius length if_collision">
         <xacro:property name="sq_r" value="${radius*radius}"/>
         <xacro:property name="sq_l" value="${length*length}"/>
@@ -36,6 +36,6 @@
                 <mass value="${mass}"/>
                 <origin xyz="0 0 0" rpy="0 0 0"/>
-                <inertia ixx="${3*sq_r*mass/12+sq_l*mass/12}" ixy="0.0" ixz="0.0" iyy="${3*sq_r*mass/12+sq_l*mass/12}"
-                iyz="0.0" izz="${mass*sq_r/2}"/>
+                <inertia ixx="${3*sq_r*arg/12+sq_l*arg/12}" ixy="0.0" ixz="0.0" iyy="${3*sq_r*arg/12+sq_l*arg/12}"
+                iyz="0.0" izz="${arg*sq_r/2}"/>
             </inertial>
             <visual>
@@ -57,5 +57,5 @@
         </link>
     </xacro:macro>
-    <xacro:macro name="rectangular_link_macro" params="suffix mass width depth height if_collision">
+    <xacro:macro name="rectangular_link_macro" params="suffix mass arg width depth height if_collision">
         <xacro:property name="sq_w" value="${width*width}"/>
         <xacro:property name="sq_d" value="${depth*depth}"/>
@@ -65,6 +65,6 @@
                 <mass value="${mass}"/>
                 <origin xyz="0 0 0" rpy="0 0 0"/>
-                <inertia ixx="${mass*sq_d/12+mass*sq_h/12}" ixy="0.0" ixz="0.0"
-                iyy="${mass*sq_w/12+mass*sq_h/12}" iyz="0.0" izz="${mass*sq_w/12+mass*sq_d/12}"/>
+                <inertia ixx="${arg*sq_d/12+arg*sq_h/12}" ixy="0.0" ixz="0.0"
+                iyy="${arg*sq_w/12+arg*sq_h/12}" iyz="0.0" izz="${arg*sq_w/12+arg*sq_d/12}"/>
             </inertial>
             <visual>
@@ -88,11 +88,11 @@
     <xacro:macro name="four_wheel_caster_macro" params="parent base_radius caster_radius z_offset">
         <xacro:property name="x" value="${base_radius*cos(pi/4)}" />
-        <xacro:sphere_macro suffix="caster1" parent="${parent}" mass="0.0001" radius="${caster_radius}" x="${x}" y="${x}" z="${z_offset}"/>
-        <xacro:sphere_macro suffix="caster2" parent="${parent}" mass="0.0001" radius="${caster_radius}" x="${-x}" y="${x}" z="${z_offset}"/>
-        <xacro:sphere_macro suffix="caster3" parent="${parent}" mass="0.0001" radius="${caster_radius}" x="${-x}" y="${-x}" z="${z_offset}"/>
-        <xacro:sphere_macro suffix="caster4" parent="${parent}" mass="0.0001" radius="${caster_radius}" x="${x}" y="${-x}" z="${z_offset}"/>
+        <xacro:sphere_macro suffix="caster1" parent="${parent}" mass="0.3" arg="3000000000.0" radius="${caster_radius}" x="${x}" y="${x}" z="${z_offset}"/>
+        <xacro:sphere_macro suffix="caster2" parent="${parent}" mass="0.3" arg="3000000000.0" radius="${caster_radius}" x="${-x}" y="${x}" z="${z_offset}"/>
+        <xacro:sphere_macro suffix="caster3" parent="${parent}" mass="0.3" arg="3000000000.0" radius="${caster_radius}" x="${-x}" y="${-x}" z="${z_offset}"/>
+        <xacro:sphere_macro suffix="caster4" parent="${parent}" mass="0.3" arg="3000000000.0" radius="${caster_radius}" x="${x}" y="${-x}" z="${z_offset}"/>
     </xacro:macro>
     <xacro:macro name="steer_macro" params="suffix parent base_radius wheel_radius wheel_offset x y z">
-        <xacro:wheel_link_macro suffix="${suffix}_base" mass="10.0" radius="${base_radius}" length="0.1" if_collision="false"/>
+        <xacro:wheel_link_macro suffix="${suffix}_base" mass="0.01" arg="10000000.0" radius="${base_radius}" length="0.1" if_collision="false"/>
         <joint name="${suffix}_base_joint" type="continuous">
             <parent link="${parent}"/>
@@ -101,5 +101,5 @@
             <axis xyz="0 0 1"/>
         </joint>
-        <xacro:wheel_link_macro suffix="${suffix}" mass="0.0001" radius="${wheel_radius}" length="0.001" if_collision="true"/>
+        <xacro:wheel_link_macro suffix="${suffix}" mass="0.0000001" arg="100.0" radius="${wheel_radius}" length="0.001" if_collision="true"/>
         <joint name="${suffix}_joint" type="continuous">
             <parent link="${suffix}_base_link"/>

Commit message: reduction model

File: auto_drive/src/holonomic_sim/models/HolonomicUrdf/model.urdf (robot description, URDF)
Before this commit: robot HolonomicUrdf, 4 links, 3 joints
Links:
- removed link wheel
- removed link wheel_base
- added link base_lidar_link, mass 0.01; visual cylinder length=0.05 radius=0.05
- added link caster1_link, mass 0.3; collision sphere radius=0.035; visual sphere radius=0.035
- added link caster2_link, mass 0.3; collision sphere radius=0.035; visual sphere radius=0.035
- added link caster3_link, mass 0.3; collision sphere radius=0.035; visual sphere radius=0.035
- added link caster4_link, mass 0.3; collision sphere radius=0.035; visual sphere radius=0.035
- added link wheel_base_link, mass 0.01
- added link wheel_link, mass 1e-07; collision cylinder length=0.001 radius=0.2
- link base_link: mass 100.0 -> 100; geometry visual box size=0.3 0.3 0.06
Joints:
- added joint base_lidar_joint: type fixed, parent base_link, child base_lidar_link, origin xyz=0.15 0 0.011 rpy=0 0 0
- added joint caster1_joint: type fixed, parent base_link, child caster1_link, origin xyz=0.15000000000000002 0.15000000000000002 -0.015 rpy=0 0 0
- added joint caster2_joint: type fixed, parent base_link, child caster2_link, origin xyz=-0.15000000000000002 0.15000000000000002 -0.015 rpy=0 0 0
- added joint caster3_joint: type fixed, parent base_link, child caster3_link, origin xyz=-0.15000000000000002 -0.15000000000000002 -0.015 rpy=0 0 0
- added joint caster4_joint: type fixed, parent base_link, child caster4_link, origin xyz=0.15000000000000002 -0.15000000000000002 -0.015 rpy=0 0 0
- joint wheel_base_joint: child wheel_base -> wheel_base_link
- joint wheel_joint: child wheel -> wheel_link; origin xyz=0 0 -0.1 rpy=-1.57 0 0 -> xyz=0 0 0.15 rpy=-1.57 0 0; parent wheel_base -> wheel_base_link

File: auto_drive/src/holonomic_sim/models/HolonomicUrdf/model.xacro (robot description, xacro)
@@ -2,6 +2,6 @@
     <xacro:include filename="$(find holonomic_sim)/models/xacro/common.xacro"/>
     <link name="base_footprint"/>
-    <xacro:property name="base_size" value="0.5"/>
-    <xacro:rectangular_link_macro suffix="base" mass="100" arg="100.0" width="${base_size}" height="${base_size/5}" depth="${base_size}" if_collision="false"/>
+    <xacro:property name="base_size" value="0.3"/>
+    <xacro:rectangular_link_macro suffix="base" mass="100" arg="10.0" width="${base_size}" height="${base_size/2}" depth="${base_size}" if_collision="false"/>
     <joint name="base_joint" type="fixed">
         <parent link="base_footprint"/>
@@ -10,5 +10,5 @@
     <xacro:steer_macro suffix="wheel" parent="base_link" base_radius="0.3" wheel_radius="0.2" x="0" y="0" z="0" wheel_offset="0.15"/>
     <xacro:four_wheel_caster_macro parent="base_link" base_radius="${sqrt(base_size/2*base_size/2*2)}" caster_radius="0.035" z_offset="-0.015"/>
-    <xacro:lidar_macro suffix="base" parent="base_link" x="0.25" y="0" z="0.031" rate="10" max_range="20" samples="270" angle="135"/>
+    <xacro:lidar_macro suffix="base" parent="base_link" x="0.15" y="0" z="0.011" rate="10" max_range="20" samples="270" angle="135"/>
     <gazebo>
         <!-- Global odometer -->
@@ -16,5 +16,5 @@
             filename="ignition-gazebo-odometry-publisher-system"
             name="ignition::gazebo::systems::OdometryPublisher">
-            <odom_publish_frequency>50</odom_publish_frequency>
+            <odom_publish_frequency>100</odom_publish_frequency>
             <odom_topic>/odom</odom_topic>
             <odom_frame>odom</odom_frame>

File: auto_drive/src/holonomic_sim/models/HolonomicUrdf/model_tx.urdf (robot description, URDF)
Before this commit: robot HolonomicUrdf, 9 links, 8 joints
Links:
- link base_lidar_link: geometry visual cylinder length=0.05 radius=0.05
- link base_link: geometry visual box size=0.5 0.5 0.1
- link caster1_link: geometry collision sphere radius=0.035; visual sphere radius=0.035
- link caster2_link: geometry collision sphere radius=0.035; visual sphere radius=0.035
- link caster3_link: geometry collision sphere radius=0.035; visual sphere radius=0.035
- link caster4_link: geometry collision sphere radius=0.035; visual sphere radius=0.035
- link wheel_base_link: geometry 
- link wheel_link: geometry collision cylinder length=0.001 radius=0.2
Joints:
- joint base_lidar_joint: origin xyz=0 0 0.5 rpy=0 0 0 -> xyz=0.15 0 0.011 rpy=0 0 0
- joint caster1_joint: origin xyz=0.5000000000000001 0.5000000000000001 -0.25 rpy=0 0 0 -> xyz=0.25000000000000006 0.25000000000000006 -0.015 rpy=0 0 0
- joint caster2_joint: origin xyz=-0.5000000000000001 0.5000000000000001 -0.25 rpy=0 0 0 -> xyz=-0.25000000000000006 0.25000000000000006 -0.015 rpy=0 0 0
- joint caster3_joint: origin xyz=-0.5000000000000001 -0.5000000000000001 -0.25 rpy=0 0 0 -> xyz=-0.25000000000000006 -0.25000000000000006 -0.015 rpy=0 0 0
- joint caster4_joint: origin xyz=0.5000000000000001 -0.5000000000000001 -0.25 rpy=0 0 0 -> xyz=0.25000000000000006 -0.25000000000000006 -0.015 rpy=0 0 0
- joint wheel_joint: origin xyz=0 0 -0.1 rpy=-1.57 0 0 -> xyz=0 0 0.15 rpy=-1.57 0 0

File: auto_drive/src/holonomic_sim/models/xacro/common.xacro (robot description, xacro)
@@ -126,11 +126,11 @@
     <xacro:macro name="four_wheel_caster_macro" params="parent base_radius caster_radius z_offset">
         <xacro:property name="x" value="${base_radius*cos(pi/4)}" />
-        <xacro:sphere_macro suffix="caster1" parent="${parent}" mass="0.3" arg="3000000000.0" radius="${caster_radius}" x="${x}" y="${x}" z="${z_offset}"/>
-        <xacro:sphere_macro suffix="caster2" parent="${parent}" mass="0.3" arg="3000000000.0" radius="${caster_radius}" x="${-x}" y="${x}" z="${z_offset}"/>
-        <xacro:sphere_macro suffix="caster3" parent="${parent}" mass="0.3" arg="3000000000.0" radius="${caster_radius}" x="${-x}" y="${-x}" z="${z_offset}"/>
-        <xacro:sphere_macro suffix="caster4" parent="${parent}" mass="0.3" arg="3000000000.0" radius="${caster_radius}" x="${x}" y="${-x}" z="${z_offset}"/>
+        <xacro:sphere_macro suffix="caster1" parent="${parent}" mass="0.3" arg="3.0" radius="${caster_radius}" x="${x}" y="${x}" z="${z_offset}"/>
+        <xacro:sphere_macro suffix="caster2" parent="${parent}" mass="0.3" arg="3.0" radius="${caster_radius}" x="${-x}" y="${x}" z="${z_offset}"/>
+        <xacro:sphere_macro suffix="caster3" parent="${parent}" mass="0.3" arg="3.0" radius="${caster_radius}" x="${-x}" y="${-x}" z="${z_offset}"/>
+        <xacro:sphere_macro suffix="caster4" parent="${parent}" mass="0.3" arg="3.0" radius="${caster_radius}" x="${x}" y="${-x}" z="${z_offset}"/>
     </xacro:macro>
     <xacro:macro name="steer_macro" params="suffix parent base_radius wheel_radius wheel_offset x y z">
-        <xacro:cylinder_link_macro suffix="${suffix}_base" mass="0.01" arg="10000000.0" radius="${base_radius}" length="0.1" if_collision="false" if_visual="false"/>
+        <xacro:cylinder_link_macro suffix="${suffix}_base" mass="0.01" arg="100.0" radius="${base_radius}" length="0.1" if_collision="false" if_visual="false"/>
         <joint name="${suffix}_base_joint" type="continuous">
             <parent link="${parent}"/>
@@ -139,5 +139,5 @@
             <axis xyz="0 0 1"/>
         </joint>
-        <xacro:cylinder_link_macro suffix="${suffix}" mass="0.0000001" arg="100.0" radius="${wheel_radius}" length="0.001" if_collision="true" if_visual="false"/>
+        <xacro:cylinder_link_macro suffix="${suffix}" mass="0.0000001" arg="1.0" radius="${wheel_radius}" length="0.001" if_collision="true" if_visual="false"/>
         <joint name="${suffix}_joint" type="continuous">
             <parent link="${suffix}_base_link"/>
