Commit message: add lidar

File: auto_drive/src/holonomic_sim/models/HolonomicUrdf/model.xacro (robot description, xacro)
@@ -10,4 +10,5 @@
     <xacro:steer_macro suffix="wheel" parent="base_link" base_radius="0.3" wheel_radius="0.2" x="0" y="0" z="0" wheel_offset="-0.1"/>
     <xacro:four_wheel_caster_macro parent="base_link" base_radius="${sqrt(base_size/2*base_size/2*2)}" caster_radius="0.05" z_offset="-0.25"/>
+    <xacro:lidar_macro suffix="base" parent="base_link" x="0" y="0" z="0.5" rate="10" range="20" samples="270" angle="135"/>
     <gazebo>
         <!-- Global odometer -->

File: auto_drive/src/holonomic_sim/models/HolonomicUrdf/model_tx.xacro (robot description, xacro)
@@ -176,4 +176,55 @@
     <parent link="base_link"/>
     <child link="caster4_link"/>
+  </joint>
+  <link name="base_lidar_link">
+    <inertial>
+      <mass value="0.01"/>
+      <origin rpy="0 0 0" xyz="0 0 0"/>
+      <inertia ixx="1.4583333333333337e-05" ixy="0.0" ixz="0.0" iyy="1.4583333333333337e-05" iyz="0.0" izz="1.2500000000000002e-05"/>
+    </inertial>
+    <visual>
+      <geometry>
+        <cylinder length="0.1" radius="0.05"/>
+      </geometry>
+      <material name="red">
+        <color rgba="1.0 0.0 0.0 1.0"/>
+      </material>
+    </visual>
+  </link>
+  <gazebo reference="base_lidar">
+    <sensor name="base" type="ray">
+      <pose>0 0 0 0 0 0</pose>
+      <visualize>true</visualize>
+      <update_rate>10</update_rate>
+      <ray>
+        <scan>
+          <horizontal>
+            <samples>400</samples>
+            <resolution>1</resolution>
+            <min_angle>-1.5707963267948966</min_angle>
+            <max_angle>1.5707963267948966</max_angle>
+          </horizontal>
+        </scan>
+        <range>
+          <min>0.10</min>
+          <max>20.0</max>
+          <resolution>0.01</resolution>
+        </range>
+        <noise>
+          <type>gaussian</type>
+          <mean>0.0</mean>
+          <stddev>0.01</stddev>
+        </noise>
+      </ray>
+      <plugin filename="libgazebo_ros_laser.so" name="gazebo_ros_lidar_controller">
+        <topicName>/base_link/scan</topicName>
+        <frameName>base_link</frameName>
+      </plugin>
+    </sensor>
+  </gazebo>
+  <joint name="base_joint" type="fixed">
+    <parent link="base_link"/>
+    <child link="base_lidar"/>
+    <origin rpy="0 0 0" xyz="0 0 0.5"/>
   </joint>
   <gazebo>

File: auto_drive/src/holonomic_sim/models/xacro/common.xacro (robot description, xacro)
@@ -29,5 +29,5 @@
         </joint>
     </xacro:macro>
-    <xacro:macro name="wheel_link_macro" params="suffix mass arg radius length if_collision">
+    <xacro:macro name="cylinder_link_macro" params="suffix mass arg radius length if_collision">
         <xacro:property name="sq_r" value="${radius*radius}"/>
         <xacro:property name="sq_l" value="${length*length}"/>
@@ -86,4 +86,35 @@
         </link>
     </xacro:macro>
+    <xacro:macro name="lidar_macro" params="suffix parent x y z rate range samples angle">
+        <xacro:cylinder_link_macro suffix="${suffix}_lidar" mass="0.01" arg="0.01" radius="0.05" length="0.1" if_collision="false"/>
+        <joint name="${suffix}_lidar_joint" type="fixed">
+            <parent link="${parent}"/>
+            <child  link="${suffix}_lidar_link"/>
+            <origin xyz="${x} ${y} ${z}" rpy="0 0 0"/>
+        </joint>
+        <gazebo reference="${suffix}_lidar_link">
+            <sensor name="gpu_lidar" type="gpu_lidar">
+                <topic>scan</topic>
+                <ignition_frame_id>base_footprint</ignition_frame_id>
+                <update_rate>${rate}</update_rate>
+                <ray>
+                  <scan>
+                    <horizontal>
+                      <samples>${samples}</samples>
+                      <resolution>1</resolution>
+                      <min_angle>${radians(angle)}</min_angle>
+                      <max_angle>${radians(-angle)}</max_angle>
+                    </horizontal>
+                  </scan>
+                  <range>
+                    <min>0.1</min>
+                    <max>${range}</max>
+                  </range>
+                </ray>
+                <always_on>true</always_on>
+                <visualize>true</visualize>
+              </sensor>
+        </gazebo>
+      </xacro:macro>
     <xacro:macro name="four_wheel_caster_macro" params="parent base_radius caster_radius z_offset">
         <xacro:property name="x" value="${base_radius*cos(pi/4)}" />
@@ -94,5 +125,5 @@
     </xacro:macro>
     <xacro:macro name="steer_macro" params="suffix parent base_radius wheel_radius wheel_offset x y z">
-        <xacro:wheel_link_macro suffix="${suffix}_base" mass="0.01" arg="10000000.0" radius="${base_radius}" length="0.1" if_collision="false"/>
+        <xacro:cylinder_link_macro suffix="${suffix}_base" mass="0.01" arg="10000000.0" radius="${base_radius}" length="0.1" if_collision="false"/>
         <joint name="${suffix}_base_joint" type="continuous">
             <parent link="${parent}"/>
@@ -101,5 +132,5 @@
             <axis xyz="0 0 1"/>
         </joint>
-        <xacro:wheel_link_macro suffix="${suffix}" mass="0.0000001" arg="100.0" radius="${wheel_radius}" length="0.001" if_collision="true"/>
+        <xacro:cylinder_link_macro suffix="${suffix}" mass="0.0000001" arg="100.0" radius="${wheel_radius}" length="0.001" if_collision="true"/>
         <joint name="${suffix}_joint" type="continuous">
             <parent link="${suffix}_base_link"/>

Commit message: update

File: auto_drive/src/holonomic_sim/models/HolonomicUrdf/model.xacro (robot description, xacro)
@@ -2,5 +2,5 @@
     <xacro:include filename="$(find holonomic_sim)/models/xacro/common.xacro"/>
     <link name="base_footprint"/>
-    <xacro:property name="base_size" value="1.0"/>
+    <xacro:property name="base_size" value="0.5"/>
     <xacro:rectangular_link_macro suffix="base" mass="100" arg="100.0" width="${base_size}" height="${base_size/2}" depth="${base_size}" if_collision="false"/>
     <joint name="base_joint" type="fixed">

Commit message: fixed

File: auto_drive/src/holonomic_sim/models/HolonomicUrdf/model.xacro (robot description, xacro)
@@ -10,5 +10,5 @@
     <xacro:steer_macro suffix="wheel" parent="base_link" base_radius="0.3" wheel_radius="0.2" x="0" y="0" z="0" wheel_offset="-0.1"/>
     <xacro:four_wheel_caster_macro parent="base_link" base_radius="${sqrt(base_size/2*base_size/2*2)}" caster_radius="0.05" z_offset="-0.25"/>
-    <xacro:lidar_macro suffix="base" parent="base_link" x="0" y="0" z="0.5" rate="10" range="20" samples="270" angle="135"/>
+    <xacro:lidar_macro suffix="base" parent="base_link" x="0" y="0" z="0.5" rate="10" max_range="20" samples="270" angle="135"/>
     <gazebo>
         <!-- Global odometer -->

File: auto_drive/src/holonomic_sim/models/xacro/common.xacro (robot description, xacro)
@@ -86,5 +86,5 @@
         </link>
     </xacro:macro>
-    <xacro:macro name="lidar_macro" params="suffix parent x y z rate range samples angle">
+    <xacro:macro name="lidar_macro" params="suffix parent x y z rate max_range samples angle">
         <xacro:cylinder_link_macro suffix="${suffix}_lidar" mass="0.01" arg="0.01" radius="0.05" length="0.1" if_collision="false"/>
         <joint name="${suffix}_lidar_joint" type="fixed">
@@ -109,5 +109,5 @@
                   <range>
                     <min>0.1</min>
-                    <max>${range}</max>
+                    <max>${max_range}</max>
                   </range>
                 </ray>

Commit message: fix lidar

File: auto_drive/src/holonomic_sim/models/HolonomicUrdf/model.xacro (robot description, xacro)
@@ -3,12 +3,12 @@
     <link name="base_footprint"/>
     <xacro:property name="base_size" value="0.5"/>
-    <xacro:rectangular_link_macro suffix="base" mass="100" arg="100.0" width="${base_size}" height="${base_size/2}" depth="${base_size}" if_collision="false"/>
+    <xacro:rectangular_link_macro suffix="base" mass="100" arg="100.0" width="${base_size}" height="${base_size/5}" depth="${base_size}" if_collision="false"/>
     <joint name="base_joint" type="fixed">
         <parent link="base_footprint"/>
         <child  link="base_link"/>
     </joint>
-    <xacro:steer_macro suffix="wheel" parent="base_link" base_radius="0.3" wheel_radius="0.2" x="0" y="0" z="0" wheel_offset="-0.1"/>
-    <xacro:four_wheel_caster_macro parent="base_link" base_radius="${sqrt(base_size/2*base_size/2*2)}" caster_radius="0.05" z_offset="-0.25"/>
-    <xacro:lidar_macro suffix="base" parent="base_link" x="0" y="0" z="0.5" rate="10" max_range="20" samples="270" angle="135"/>
+    <xacro:steer_macro suffix="wheel" parent="base_link" base_radius="0.3" wheel_radius="0.2" x="0" y="0" z="0" wheel_offset="0.15"/>
+    <xacro:four_wheel_caster_macro parent="base_link" base_radius="${sqrt(base_size/2*base_size/2*2)}" caster_radius="0.035" z_offset="-0.015"/>
+    <xacro:lidar_macro suffix="base" parent="base_link" x="0.25" y="0" z="0.031" rate="10" max_range="20" samples="270" angle="135"/>
     <gazebo>
         <!-- Global odometer -->

File: auto_drive/src/holonomic_sim/models/xacro/common.xacro (robot description, xacro)
@@ -29,5 +29,5 @@
         </joint>
     </xacro:macro>
-    <xacro:macro name="cylinder_link_macro" params="suffix mass arg radius length if_collision">
+    <xacro:macro name="cylinder_link_macro" params="suffix mass arg radius length if_collision if_visual">
         <xacro:property name="sq_r" value="${radius*radius}"/>
         <xacro:property name="sq_l" value="${length*length}"/>
@@ -39,12 +39,14 @@
                 iyz="0.0" izz="${arg*sq_r/2}"/>
             </inertial>
-            <visual>
-                <geometry>
-                    <cylinder length="${length}" radius="${radius}"/>
-                </geometry>
-                <material name="red">
-                    <color rgba="1.0 0.0 0.0 1.0"/>
-                </material>
-            </visual>
+            <xacro:if value="${if_visual}">
+                <visual>
+                    <geometry>
+                        <cylinder length="${length}" radius="${radius}"/>
+                    </geometry>
+                    <material name="red">
+                        <color rgba="1.0 0.0 0.0 1.0"/>
+                    </material>
+                </visual>
+            </xacro:if>
             <xacro:if value="${if_collision}">
                 <collision>
@@ -87,5 +89,5 @@
     </xacro:macro>
     <xacro:macro name="lidar_macro" params="suffix parent x y z rate max_range samples angle">
-        <xacro:cylinder_link_macro suffix="${suffix}_lidar" mass="0.01" arg="0.01" radius="0.05" length="0.1" if_collision="false"/>
+        <xacro:cylinder_link_macro suffix="${suffix}_lidar" mass="0.01" arg="0.01" radius="0.05" length="0.05" if_collision="false"  if_visual="true"/>
         <joint name="${suffix}_lidar_joint" type="fixed">
             <parent link="${parent}"/>
@@ -95,6 +97,6 @@
         <gazebo reference="${suffix}_lidar_link">
             <sensor name="gpu_lidar" type="gpu_lidar">
-                <topic>scan</topic>
-                <ignition_frame_id>base_footprint</ignition_frame_id>
+                <topic>/scan</topic>
+                <ignition_frame_id>${suffix}_lidar_link</ignition_frame_id>
                 <update_rate>${rate}</update_rate>
                 <ray>
@@ -103,10 +105,10 @@
                       <samples>${samples}</samples>
                       <resolution>1</resolution>
-                      <min_angle>${radians(angle)}</min_angle>
-                      <max_angle>${radians(-angle)}</max_angle>
+                      <min_angle>${-radians(angle)}</min_angle>
+                      <max_angle>${radians(angle)}</max_angle>
                     </horizontal>
                   </scan>
                   <range>
-                    <min>0.1</min>
+                    <min>0.01</min>
                     <max>${max_range}</max>
                   </range>
@@ -125,5 +127,5 @@
     </xacro:macro>
     <xacro:macro name="steer_macro" params="suffix parent base_radius wheel_radius wheel_offset x y z">
-        <xacro:cylinder_link_macro suffix="${suffix}_base" mass="0.01" arg="10000000.0" radius="${base_radius}" length="0.1" if_collision="false"/>
+        <xacro:cylinder_link_macro suffix="${suffix}_base" mass="0.01" arg="10000000.0" radius="${base_radius}" length="0.1" if_collision="false" if_visual="false"/>
         <joint name="${suffix}_base_joint" type="continuous">
             <parent link="${parent}"/>
@@ -132,5 +134,5 @@
             <axis xyz="0 0 1"/>
         </joint>
-        <xacro:cylinder_link_macro suffix="${suffix}" mass="0.0000001" arg="100.0" radius="${wheel_radius}" length="0.001" if_collision="true"/>
+        <xacro:cylinder_link_macro suffix="${suffix}" mass="0.0000001" arg="100.0" radius="${wheel_radius}" length="0.001" if_collision="true" if_visual="false"/>
         <joint name="${suffix}_joint" type="continuous">
             <parent link="${suffix}_base_link"/>

Commit message: update model

File: auto_drive/src/holonomic_sim/models/HolonomicUrdf/model.xacro (robot description, xacro)
@@ -3,5 +3,5 @@
     <link name="base_footprint"/>
     <xacro:property name="base_size" value="0.3"/>
-    <xacro:rectangular_link_macro suffix="base" mass="100" arg="10.0" width="${base_size}" height="${base_size/2}" depth="${base_size}" if_collision="false"/>
+    <xacro:rectangular_link_macro suffix="base" mass="0.0001" arg="0.0001" width="${base_size}" height="${base_size/2}" depth="${base_size}" if_collision="false" if_visual="false"/>
     <joint name="base_joint" type="fixed">
         <parent link="base_footprint"/>
@@ -29,5 +29,6 @@
         <plugin filename="libHolonomicPlugin.so" name="holonomic_sim::HolonomicPlugin">
             <wheel_joint>wheel_joint</wheel_joint>
-            <base_joint>wheel_base_joint</base_joint>
+            <top_base_joint>bottom_wheel_base_joint</top_base_joint>
+            <bottom_base_joint>top_wheel_base_joint</bottom_base_joint>
         </plugin>
     </gazebo>

File: auto_drive/src/holonomic_sim/models/xacro/common.xacro (robot description, xacro)
@@ -59,5 +59,5 @@
         </link>
     </xacro:macro>
-    <xacro:macro name="rectangular_link_macro" params="suffix mass arg width depth height if_collision">
+    <xacro:macro name="rectangular_link_macro" params="suffix mass arg width depth height if_collision if_visual">
         <xacro:property name="sq_w" value="${width*width}"/>
         <xacro:property name="sq_d" value="${depth*depth}"/>
@@ -70,12 +70,14 @@
                 iyy="${arg*sq_w/12+arg*sq_h/12}" iyz="0.0" izz="${arg*sq_w/12+arg*sq_d/12}"/>
             </inertial>
-            <visual>
-                <geometry>
-                    <box size="${width} ${depth} ${height}"/>
-                </geometry>
-                <material name="blue">
-                    <color rgba="0.0 0.0 1.0 1.0"/>
-                </material>
-            </visual>
+            <xacro:if value="${if_visual}">
+                <visual>
+                    <geometry>
+                        <box size="${width} ${depth} ${height}"/>
+                    </geometry>
+                    <material name="blue">
+                        <color rgba="0.0 0.0 1.0 1.0"/>
+                    </material>
+                </visual>
+            </xacro:if>
             <xacro:if value="${if_collision}">
                 <collision>
@@ -89,5 +91,5 @@
     </xacro:macro>
     <xacro:macro name="lidar_macro" params="suffix parent x y z rate max_range samples angle">
-        <xacro:cylinder_link_macro suffix="${suffix}_lidar" mass="0.01" arg="0.01" radius="0.05" length="0.05" if_collision="false"  if_visual="true"/>
+        <xacro:cylinder_link_macro suffix="${suffix}_lidar" mass="0.0001" arg="0.0001" radius="0.05" length="0.05" if_collision="false"  if_visual="true"/>
         <joint name="${suffix}_lidar_joint" type="fixed">
             <parent link="${parent}"/>
@@ -126,20 +128,27 @@
     <xacro:macro name="four_wheel_caster_macro" params="parent base_radius caster_radius z_offset">
         <xacro:property name="x" value="${base_radius*cos(pi/4)}" />
-        <xacro:sphere_macro suffix="caster1" parent="${parent}" mass="0.3" arg="3.0" radius="${caster_radius}" x="${x}" y="${x}" z="${z_offset}"/>
-        <xacro:sphere_macro suffix="caster2" parent="${parent}" mass="0.3" arg="3.0" radius="${caster_radius}" x="${-x}" y="${x}" z="${z_offset}"/>
-        <xacro:sphere_macro suffix="caster3" parent="${parent}" mass="0.3" arg="3.0" radius="${caster_radius}" x="${-x}" y="${-x}" z="${z_offset}"/>
-        <xacro:sphere_macro suffix="caster4" parent="${parent}" mass="0.3" arg="3.0" radius="${caster_radius}" x="${x}" y="${-x}" z="${z_offset}"/>
+        <xacro:sphere_macro suffix="caster1" parent="${parent}" mass="0.003" arg="0.00003" radius="${caster_radius}" x="${x}" y="${x}" z="${z_offset}"/>
+        <xacro:sphere_macro suffix="caster2" parent="${parent}" mass="0.003" arg="0.00003" radius="${caster_radius}" x="${-x}" y="${x}" z="${z_offset}"/>
+        <xacro:sphere_macro suffix="caster3" parent="${parent}" mass="0.003" arg="0.00003" radius="${caster_radius}" x="${-x}" y="${-x}" z="${z_offset}"/>
+        <xacro:sphere_macro suffix="caster4" parent="${parent}" mass="0.003" arg="0.00003" radius="${caster_radius}" x="${x}" y="${-x}" z="${z_offset}"/>
     </xacro:macro>
     <xacro:macro name="steer_macro" params="suffix parent base_radius wheel_radius wheel_offset x y z">
-        <xacro:cylinder_link_macro suffix="${suffix}_base" mass="0.01" arg="100.0" radius="${base_radius}" length="0.1" if_collision="false" if_visual="false"/>
-        <joint name="${suffix}_base_joint" type="continuous">
+        <xacro:cylinder_link_macro suffix="top_${suffix}_base" mass="10000.0" arg="1000000.0" radius="${base_radius}" length="0.001" if_collision="false" if_visual="true"/>
+        <joint name="top_${suffix}_base_joint" type="continuous">
             <parent link="${parent}"/>
-            <child  link="${suffix}_base_link"/>
-            <origin xyz="${x} ${y} ${z}" rpy="0 0 0"/>
+            <child  link="top_${suffix}_base_link"/>
+            <origin xyz="${x} ${y} ${z+0.1}" rpy="0 0 0"/>
             <axis xyz="0 0 1"/>
         </joint>
-        <xacro:cylinder_link_macro suffix="${suffix}" mass="0.0000001" arg="1.0" radius="${wheel_radius}" length="0.001" if_collision="true" if_visual="false"/>
+        <xacro:cylinder_link_macro suffix="bottom_${suffix}_base" mass="1.0" arg="1.0" radius="${base_radius}" length="0.001" if_collision="false" if_visual="true"/>
+        <joint name="bottom_${suffix}_base_joint" type="continuous">
+            <parent link="top_${suffix}_base_link"/>
+            <child  link="bottom_${suffix}_base_link"/>
+            <origin xyz="${x} ${y} ${z-0.1}" rpy="0 0 0"/>
+            <axis xyz="0 0 1"/>
+        </joint>
+        <xacro:cylinder_link_macro suffix="${suffix}" mass="0.1" arg="0.1" radius="${wheel_radius}" length="0.001" if_collision="true" if_visual="true"/>
         <joint name="${suffix}_joint" type="continuous">
-            <parent link="${suffix}_base_link"/>
+            <parent link="bottom_${suffix}_base_link"/>
             <child  link="${suffix}_link"/>
             <origin xyz="0 0 ${wheel_offset}" rpy="-1.57 0 0"/>

Commit message: create accurate map

File: auto_drive/src/holonomic_sim/models/HolonomicUrdf/model.xacro (robot description, xacro)
@@ -10,5 +10,5 @@
     <xacro:steer_macro suffix="wheel" parent="base_link" base_radius="0.3" wheel_radius="0.2" x="0" y="0" z="0" wheel_offset="0.15"/>
     <xacro:four_wheel_caster_macro parent="base_link" base_radius="${sqrt(base_size/2*base_size/2*2)}" caster_radius="0.035" z_offset="-0.015"/>
-    <xacro:lidar_macro suffix="base" parent="base_link" x="0.15" y="0" z="0.025" rate="20" max_range="20" samples="270" angle="135"/>
+    <xacro:lidar_macro suffix="base" parent="base_link" x="0.15" y="0" z="0.025" rate="20" max_range="20" samples="270" angle="135" noise="0.01"/>
     <gazebo>
         <!-- Global odometer -->

File: auto_drive/src/holonomic_sim/models/xacro/common.xacro (robot description, xacro)
@@ -93,5 +93,5 @@
     </xacro:macro>
     <!-- lidar macro with lidar plugin for ign gz-->
-    <xacro:macro name="lidar_macro" params="suffix parent x y z rate max_range samples angle">
+    <xacro:macro name="lidar_macro" params="suffix parent x y z rate max_range samples angle noise">
         <xacro:cylinder_link_macro suffix="${suffix}_lidar" mass="0.0001" arg="0.0001" radius="0.05" length="0.05" if_collision="false"  if_visual="true"/>
         <joint name="${suffix}_lidar_joint" type="fixed">
@@ -121,5 +121,5 @@
                     <type>gaussian</type>
                     <mean>0.0</mean>
-                    <stddev>0.0</stddev>
+                    <stddev>${noise}</stddev>
                   </noise>
                 </ray>
